File: Dummy Bridge Board.sch (EAGLE design)
At the start: 90 parts, among them J2 5787834-1, U14 ADUM3160BRWZ-RL, U22 PDS1-S5-S5-M-TR, U28 FT4232HL, U29 SN74HC595DR, U30 LP5907MFX-3.3/NOPB, U9 TPS54540DDARQ1, Y2 CX3225GB12000P0HPQCC

Commit message: DONE- added vert banana sockets
Parts:
- removed H1: 0.1" Jumper, FormE:GENERIC_BLOCK
- removed JP11, JP23: (no value), pinhead:PINHD-1X2/90
- removed R31, R32: 1k, rcl:R-US_R0603
- removed R71: 0.007, adafruit:R-US_R0805
- added B1: BKCT2228-2-ND, FormE:CT2228
- added B2: BKCT2228-0-ND, FormE:CT2228
- added D5: PMEG3030EP,115, FormE:PMEG3030EP,115
- added H2: CARCONTROLLER-REF, FormE:CARCONTROLLER-REF
- ARX, ATX, BRX, BTX, CRX, CTX, DRX, DTX: PARTNO (none) -> 598-8130-107F
- R48, R54, R55, R56, R57, R58, R59, R60: PARTNO (none) -> ERJ-3EKF1001V
- U22: PARTNO (none) -> PDS1-S5-S5-M-TR
- U28: PARTNO (none) -> FT4232HL-REEL
- U29: PARTNO (none) -> SN74HC595DR
- U30: PARTNO (none) -> LP5907MFX-3.3/NOPB
- Y2: PARTNO (none) -> CX3225GB12000P0HPQCC
- renumbered LED10 to DTX, LED11 to DRX, LED4 to ATX, LED5 to ARX, LED6 to BTX, LED7 to BRX, LED8 to CTX, LED9 to CRX
Connections:
- removed net !PD: H4.!PD!
- removed net !POR: H4.!POR!
- removed net 5V_CURRENT_SENSE+: C89.1, C90.1, C91.1, L7.P$2, R71.1
- removed net 5V_CURRENT_SENSE-: JP11.1, R62.2, R71.2
- removed net N$16: JP23.1, R32.2
- removed net N$6: JP23.2, R31.2
- new net N$2: B1.P$1, D5.A
- net +5V: now also C89.1, C90.1, C91.1, L7.P$2, R62.2; no longer JP11.2
- net GND: now also B2.P$1
- net UART_RX1: now also H4.UART_RX1; no longer R31.1
- net UART_TX1: now also H4.UART_TX1; no longer R32.1
- net VCC: now also D5.K
Other:
- note added: "Bench Power Card"
- note removed: "?"
- note removed: "Banana Plug Socket: http://www.newark.com/multicomp/24-243-2/pcb-socket-4mm-black/dp/80P3613?CMP=KNC-GUSA-GEN-SHOPPING-NEW-MULTICOMP&ad=81605889141&gclid=Cj0KEQjw3ZS-BRD1xu3qw8uS2s4BEiQA2bcfM2f0TZ8AKgQw3kR3UXGrkgP2GbVFHKcRCi6CVmOGPdsaAl2l8P8HAQ"
- note removed: "Dummy Bridge Card"
- moved on the sheet: H4

Commit message: Added BOM
Parts:
- B1: PARTNO (none) -> CT2228-2
- B2: PARTNO (none) -> CT2228-0
Changed lines of the file:
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@@
 <attribute name="PARTNO" value="PMEG3030EP,115"/>
 </part>
-<part name="B1" library="FormE" deviceset="CT2228" device="" value="BKCT2228-2-ND"/>
-<part name="B2" library="FormE" deviceset="CT2228" device="" value="BKCT2228-0-ND"/>
+<part name="B1" library="FormE" deviceset="CT2228" device="" value="BKCT2228-2-ND">
+<attribute name="PARTNO" value="CT2228-2"/>
+</part>
+<part name="B2" library="FormE" deviceset="CT2228" device="" value="BKCT2228-0-ND">
+<attribute name="PARTNO" value="CT2228-0"/>
+</part>
 </parts>
 <sheets>
@@
 <attribute name="PARTNO" x="558.8" y="261.62" size="1.778" layer="96" rot="R90" display="off"/>
 </instance>
-<instance part="B1" gate="G$1" x="548.64" y="254" rot="R270"/>
-<instance part="B2" gate="G$1" x="548.64" y="246.38" rot="R270"/>
+<instance part="B1" gate="G$1" x="548.64" y="254" rot="R270">
+<attribute name="PARTNO" x="548.64" y="254" size="6.4516" layer="96" display="off"/>
+</instance>
+<instance part="B2" gate="G$1" x="548.64" y="246.38" rot="R270">
+<attribute name="PARTNO" x="548.64" y="246.38" size="6.4516" layer="96" display="off"/>
+</instance>
 </instances>
 <busses>

Commit message: Added Voltage supervisor, about to finish BOM
Parts:
- added C43, C73, C74: 0.1uF, rcl:C-USC0603K
- added C75, C76: 1uF, rcl:C-USC0603K
- added R61, R65: 10k, rcl:R-US_R0603
- added R63: 100, rcl:R-US_R0603
- added S2: TE-FSM4JSMATR, FormE:TE-FSM4JSMATR
- added TP26, TP27, TP28: PTR1TP20R, testpad:PTR1TP20R
- added U21: CD4050BD, FormE:CD4050BD
- added U49: TL7712A-SOIC, FormE:TL7709A-SOIC
Connections:
- new net !POR: H4.!POR!, TP28.TP, U21F.OUT
- new net +3V3: C43.1, U21POWER.VCC
- new net MAN_RESET_SIGNAL: C76.1, R63.1, R65.1, TP27.TP, U49.*RESIN
- new net N$60: R61.1, TP26.TP, U21F.IN, U49.*RESET
- new net N$72: C74.1, U49.REF
- new net N$73: C73.1, U49.CT
- new net N$74: R63.2, S2.1, S2.2
- net GND: now also C43.2, C73.2, C74.2, C75.2, C76.2, S2.3, S2.4, U21POWER.GND, U49.GND
- net VCC: now also C75.1, R61.2, R65.2, U49.SENSE, U49.VCC
Other:
- note added: "Voltage Supervisor"
- moved on the sheet: B1, B2, D5, H2, H4

Commit message: Added +3V3 Buck and finished BOM- Ready to order
Parts:
- added C40: 4.7uF, rcl:C-USC0603K
- added C70: 10uF, rcl:C-USC0603K
- added L5: 2.2uH, FormE:L0805
- added LED2: GREEN, FormE:LEDCHIP-LED0805
- added R36: 1k, rcl:R-US_R0603
- added U16: LM3671MF-3.3/NOPB, FormE:LM3671MF
Connections:
- new net N$56: LED2.C, R36.2
- new net N$57: L5.P$1, U16.SW
- net +3V3: now also C70.1, L5.P$2, LED2.A, U16.FB
- net +5V: now also C40.1, U16.EN, U16.VIN
- net GND: now also C40.2, C70.2, R36.1, U16.GND
Other:
- note added: "+3V3 Buck Converter"
- note added: "+3v3 buck"
- note added: "74479775222"
- moved on the sheet: B1, B2, D5, H2, H4

Commit message: Fixed numerous errors in BOM with wrong part values and packages
Parts:
- C42: PARTNO GRM216R71H123KA01D -> GRM188R71H123KA01D
- C43, C73, C74, C86: PARTNO GRM21BR71E104KA01L -> GRM188R71E104KA01D
- C47, C48, C50, C63, C65: PARTNO GRM188R71E104KA01D -> GRM188R61C475KAAJD
- C60, C61: PARTNO GRM188R71E104KA01D -> GRM1885C1H180JA01D
- C70, C90, C91: PARTNO GRM21BR61E106KA73L -> EMK107BBJ106MA-T
- C75, C76: PARTNO EMK212B7105KG-T -> GRM188R71E104KA01D
- C85: PARTNO CL21C090CBANNNC -> GRM1885C1H9R0DA01D
- L2, L3, L4: PARTNO BLM21PG221SN1D -> BLM21AG601SN1D
- R35: PARTNO ERJ-3EKF24R0V -> ERJ-3EKF1202V
- R36, R7: PARTNO ERJ-6ENF1001V -> ERJ-3EKF1001V
- R37, R38, R39, R40, R41, R44, R45, R46: PARTNO ERJ-3EKF24R0V -> ERJ-3EKF3300V
- R42: PARTNO ERJ-6ENF1623V -> ERJ-3EKF1623V
- R47: PARTNO ERJ-3EKF24R0V -> ERJ-3EKF1002V
- R49: PARTNO ERJ-6ENF1502V -> ERJ-3EKF1502V
- R61, R65: PARTNO ERJ-6ENF1002V -> ERJ-3EKF1002V
- R62: PARTNO ERJ-6ENF6042V -> ERJ-3EKF6042V
- R63: PARTNO ERJ-6ENF1000V -> ERJ-3EKF1000V
- R68: PARTNO ERJ-6ENF1152V -> ERJ-3EKF1152V
